File: file5FD25DF8.sch (KiCad schematic (older format))
At the start: 11 parts, among them J1 Screw_Terminal_01x02, U1 TPSM84209RKHT

Commit message: Change PS to SMPS 5v, LDO 3.3V
Parts:
- removed C1, C3: C3216X6S1V106K160AC, CAPC3216X180N, symbol C3216X6S1V106K160AC:C3216X6S1V106K160AC
- removed C2: EEE-FK1E330P, CAPAE660X610N, symbol EEE-FK1E330P:EEE-FK1E330P
- removed C4: GRM033R71E331KA01D, CAPC0603X33N, symbol GRM033R71E331KA01D:GRM033R71E331KA01D
- removed C5: GRM32ER61A107ME20L, CAPC3225X270N, symbol GRM32ER61A107ME20L:GRM32ER61A107ME20L
- removed L1: LQM18PNR47NC0L, INDC1608X55N, symbol LQM18PNR47NC0L:LQM18PNR47NC0L
- removed R3: RC0603FR-072K2L, RESC1608X55N, symbol RC0603FR-072K2L:RC0603FR-072K2L
- removed U1: TPSM84209RKHT, VREG_TPSM84209RKHT, symbol TPSM84209RKHT:TPSM84209RKHT
- added C1: GRM21BC71E475KE11L, CAPC2012X145N, symbol GRM21BC71E475KE11L:GRM21BC71E475KE11L
- added C2: 25SVPF27MX, CAPAE530X600N, symbol 25SVPF27MX:25SVPF27MX
- added C26, C28: 100nF, symbol Device:C
- added C27, C5: 1uF_X5R, symbol Device:C
- added C3: C3216X5R1H106K160AB, CAPC3216X180N, symbol C3216X5R1H106K160AB:C3216X5R1H106K160AB
- added C4: GRM32EC81C476KE15L, CAPC3225X270N, symbol GRM32EC81C476KE15L:GRM32EC81C476KE15L
- added D1: LED GREEN, symbol Device:LED
- added IC1: LD39100PU33R, SON95P300X300X100-7N-D, symbol LD39100PU33R:LD39100PU33R
- added L1: NLCV32T-R33M-EFR, IND_NLCV32T-R33M-PFR, symbol NLCV32T-R33M-PFR:NLCV32T-R33M-PFR
- added R10: 1K, symbol Device:R_Small_US
- added R3: 100k, symbol Device:R_Small_US
- added R4: CRCW04022K49FKED, RESC1005X40N, symbol CRCW04022K49FKED:CRCW04022K49FKED
- added U1: TPSM53604RDAR, B3QFN14_RDA_TEX, symbol 2020-12-12_03-26-08:TPSM53604RDAR
Connections:
- net GND: now also C1.2, C2.2, C26.2, C27.2, C28.2, C3.2, C4.2, C5.2, D1.1 (K), IC1.2 (GND), IC1.7 (EP), R4.2, U1.10 (NC), U1.11 (NC), U1.12 (AGND), U1.15 (PGND), U1.3 (NC)
- net VDD: now also C27.1, C28.1, IC1.4 (VOUT); no longer R2.1
- net at R2.2: now also R4.1, U1.9 (FB)
- net at R1.1: now also C3.1, L1.2, U1.1 (VIN), U1.14 (VIN), U1.2 (EN)
- net at J1.2 (Pin_2): now also C1.1, L1.1
- net at R1.2: now also C2.1
- new net: R3.1, U1.13 (V5V)
- new net: R3.2, U1.6 (PGOOD)
- new net: D1.2 (A), R10.2
- new net +5V: C26.1, C4.1, C5.1, IC1.1 (EN), IC1.6 (VIN), R10.1, R2.1, U1.7 (VOUT), U1.8 (VOUT)
- no-connect marks 3 -> 5
Other:
- moved on the sheet: J1, R1, R2
