File: kicad/file5FDA5731.sch (KiCad schematic (older format))
At the start: 99 parts, among them J4 Screw_Terminal_01x02, M1 BSC014N04LSI, M11 BSC014N04LSI, M12 BSC010N04LSI, M13 BSC015NE2LS5I, M14 BSC009NE2LS5I, M15 BSC014N04LSI, M17 BSC015NE2LS5I, M2 BSC010N04LSI, M3 BSC015NE2LS5I, M4 BSC009NE2LS5I, M5 BSC014N04LSI, M7 BSC015NE2LS5I, U1 LT8390AHUFD#PBF, U2 LT8390AHUFD#PBF, U3 LTC6908HS6-2TRPBF

Commit message: Adjust component values for 13.8V; add RUNSTOP driver
Parts:
- added J?: Screw_Terminal_01x02, symbol Connector:Screw_Terminal_01x02
- added Q?: BSS138L, SOT96P237X111-3N, symbol SamacSys_Parts:BSS138L
- R16, R34: value 309K, 150kHz -> 309K
- R39: value 549K -> 638K
Connections:
- net GND: now also J?.1 (Pin_1), Q?.2
- net VREG: now also J?.2 (Pin_2)
- net ENUVLO renamed U1ENUVLO
- net U1ENUVLO: now also Q?.3
- net U1ISMON renamed ISMON
- new net RUNSTOP: Q?.1
Other:
- note added: "+3V3 to\ndisable regulator"
- note added: "150kHz"
- moved on the sheet: J4
Changed lines of the file:
@@
 L Connector:Screw_Terminal_01x02 J4
 U 1 1 5FDC6F74
-P 900 10050
-F 0 "J4" H 818 9725 50  0000 C CNN
-F 1 "Screw_Terminal_01x02" H 818 9816 50  0000 C CNN
-F 2 "" H 900 10050 50  0001 C CNN
-F 3 "~" H 900 10050 50  0001 C CNN
-	1    900  10050
+P 1000 4900
+F 0 "J4" H 918 4575 50  0000 C CNN
+F 1 "Screw_Terminal_01x02" H 918 4666 50  0000 C CNN
+F 2 "" H 1000 4900 50  0001 C CNN
+F 3 "~" H 1000 4900 50  0001 C CNN
+	1    1000 4900
 	-1   0    0    1
 $EndComp
-$Comp
-L power:GND #PWR09
-U 1 1 5FDC7975
-P 1100 10250
-F 0 "#PWR09" H 1100 10000 50  0001 C CNN
-F 1 "GND" H 1105 10077 50  0000 C CNN
-F 2 "" H 1100 10250 50  0001 C CNN
-F 3 "" H 1100 10250 50  0001 C CNN
-	1    1100 10250
-	1    0    0    -1
-$EndComp
-Text Label 1300 9950 0    50   ~ 0
+Text Label 1400 4800 0    50   ~ 0
 Vin
 Wire Wire Line
-	1100 9950 1300 9950
-Wire Wire Line
-	1100 10050 1100 10250
+	1200 4800 1400 4800
 Text Label 850  1300 0    50   ~ 0
 Vin
@@
 P 9300 3250
 F 0 "R16" V 9095 3250 50  0000 C CNN
-F 1 "309K, 150kHz" V 9186 3250 50  0000 C CNN
+F 1 "309K" V 9186 3250 50  0000 C CNN
 F 2 "" H 9300 3250 50  0001 C CNN
 F 3 "~" H 9300 3250 50  0001 C CNN
@@
 P 9400 8200
 F 0 "R34" V 9195 8200 50  0000 C CNN
-F 1 "309K, 150kHz" V 9286 8200 50  0000 C CNN
+F 1 "309K" V 9286 8200 50  0000 C CNN
 F 2 "" H 9400 8200 50  0001 C CNN
 F 3 "~" H 9400 8200 50  0001 C CNN
@@
 P 15100 6250
 F 0 "R39" H 15168 6296 50  0000 L CNN
-F 1 "549K" H 15168 6205 50  0000 L CNN
+F 1 "638K" H 15168 6205 50  0000 L CNN
 F 2 "" H 15100 6250 50  0001 C CNN
 F 3 "~" H 15100 6250 50  0001 C CNN
@@
 Text Label 8400 7700 0    50   ~ 0
 U3OUT1
-Text HLabel 15900 8300 2    50   BiDi ~ 0
-ENUVLO
-Text Label 15750 8200 2    50   ~ 0
+Text HLabel 15850 8150 2    50   Input ~ 0
+RUNSTOP
+Text Label 14800 7650 2    50   ~ 0
 U1ENUVLO
-Text Label 15750 8450 2    50   ~ 0
+Text Label 14800 7900 2    50   ~ 0
 U2ENUVLO
 Wire Wire Line
-	15750 8200 15750 8300
-Wire Wire Line
-	15900 8300 15750 8300
-Connection ~ 15750 8300
-Wire Wire Line
-	15750 8300 15750 8450
-Wire Wire Line
 	3450 1300 3750 1300
 Connection ~ 3450 2750
@@
 VREG
 Wire Wire Line
-	15100 6050 15900 6050
+	15100 6050 15700 6050
 Connection ~ 15100 6050
 Text Notes 15700 6300 0    50   ~ 0
 13.8V (ADJ.)\n50A
+$Comp
+L Connector:Screw_Terminal_01x02 J?
+U 1 1 5FE78396
+P 16150 5600
+F 0 "J?" H 16068 5275 50  0000 C CNN
+F 1 "Screw_Terminal_01x02" H 16068 5366 50  0000 C CNN
+F 2 "" H 16150 5600 50  0001 C CNN
+F 3 "~" H 16150 5600 50  0001 C CNN
+	1    16150 5600
+	1    0    0    1
+$EndComp
+$Comp
+L power:GND #PWR?
+U 1 1 5FE78DFA
+P 15950 5650
+F 0 "#PWR?" H 15950 5400 50  0001 C CNN
+F 1 "GND" H 15955 5477 50  0000 C CNN
+F 2 "" H 15950 5650 50  0001 C CNN
+F 3 "" H 15950 5650 50  0001 C CNN
+	1    15950 5650
+	1    0    0    -1
+$EndComp
+Wire Wire Line
+	15950 5600 15950 5650
+Wire Wire Line
+	15950 5500 15700 5500
+Wire Wire Line
+	15700 5500 15700 6050
+Connection ~ 15700 6050
+Wire Wire Line
+	15700 6050 15900 6050
+Wire Wire Line
+	1200 4900 1200 4950
+$Comp
+L power:GND #PWR09
+U 1 1 5FDC7975
+P 1200 4950
+F 0 "#PWR09" H 1200 4700 50  0001 C CNN
+F 1 "GND" H 1205 4777 50  0000 C CNN
+F 2 "" H 1200 4950 50  0001 C CNN
+F 3 "" H 1200 4950 50  0001 C CNN
+	1    1200 4950
+	1    0    0    -1
+$EndComp
+Text Label 15750 7550 2    50   ~ 0
+U1ISMON
+Text HLabel 15950 7550 2    50   Output ~ 0
+ISMON
+Wire Wire Line
+	15750 7550 15950 7550
+Text Notes 9450 3400 1    50   ~ 0
+150kHz
+Text Notes 9550 8350 1    50   ~ 0
+150kHz
+$Comp
+L SamacSys_Parts:BSS138L Q?
+U 1 1 602C5287
+P 15750 8150
+F 0 "Q?" H 16179 8296 50  0000 L CNN
+F 1 "BSS138L" H 16179 8205 50  0000 L CNN
+F 2 "SOT96P237X111-3N" H 16200 8100 50  0001 L CNN
+F 3 "https://www.onsemi.com/products/discretes-drivers/mosfets/bss138l" H 16200 8000 50  0001 L CNN
+F 4 "ON SEMICONDUCTOR/FAIRCHILD - BSS138L - MOSFET, N-CHANNEL, 50V, 0.2A, SOT-23-3" H 16200 7900 50  0001 L CNN "Description"
+F 5 "1.11" H 16200 7800 50  0001 L CNN "Height"
+F 6 "ON Semiconductor" H 16200 7700 50  0001 L CNN "Manufacturer_Name"
+F 7 "BSS138L" H 16200 7600 50  0001 L CNN "Manufacturer_Part_Number"
+F 8 "BSS138L" H 16200 7500 50  0001 L CNN "Arrow Part Number"
+F 9 "https://www.arrow.com/en/products/bss138l/on-semiconductor" H 16200 7400 50  0001 L CNN "Arrow Price/Stock"
+F 10 "512-BSS138L" H 16200 7300 50  0001 L CNN "Mouser Part Number"
+F 11 "https://www.mouser.co.uk/ProductDetail/ON-Semiconductor-Fairchild/BSS138L/?qs=C8E66ftkQtxfAHmiWaRE%252Bg%3D%3D" H 16200 7200 50  0001 L CNN "Mouser Price/Stock"
+	1    15750 8150
+	-1   0    0    -1
+$EndComp
+Wire Wire Line
+	14800 7650 14800 7750
+Wire Wire Line
+	15450 7750 14800 7750
+Connection ~ 14800 7750
+Wire Wire Line
+	14800 7750 14800 7900
+$Comp
+L power:GND #PWR?
+U 1 1 603D8582
+P 15450 8400
+F 0 "#PWR?" H 15450 8150 50  0001 C CNN
+F 1 "GND" H 15455 8227 50  0000 C CNN
+F 2 "" H 15450 8400 50  0001 C CNN
+F 3 "" H 15450 8400 50  0001 C CNN
+	1    15450 8400
+	1    0    0    -1
+$EndComp
+Wire Wire Line
+	15750 8150 15850 8150
+Wire Wire Line
+	15450 8350 15450 8400
+Text Notes 16250 8350 2    50   ~ 0
++3V3 to\ndisable regulator
 $EndSCHEMATC

Commit message: Sense resistors Section 1
Parts:
- added R? (x2): KRL6432D-M-R006-G-T1, RESC3163X50N, symbol SamacSys_Parts:KRL6432E-C-R006-F-T1
Connections:
- net U1VOUT: now also R?.1, R?.1
- net VREG: now also R?.2, R?.2
Changed lines of the file:
@@
 Wire Wire Line
 	13200 6550 13350 6550
-Wire Wire Line
-	15300 1100 15300 5300
-Wire Wire Line
-	15300 5300 13600 5300
-Wire Wire Line
-	13600 5300 13600 6050
 Text Label 7550 8900 3    50   ~ 0
 U1ISMON
@@
 Text Notes 16250 8350 2    50   ~ 0
 +3V3 to\ndisable regulator
+Wire Wire Line
+	13600 3100 13600 6050
+Wire Wire Line
+	15300 1100 15300 3100
+Wire Wire Line
+	15300 3100 13600 3100
+$Comp
+L SamacSys_Parts:KRL6432E-C-R006-F-T1 R?
+U 1 1 5FFA054E
+P 14100 5200
+F 0 "R?" H 14450 5425 50  0000 C CNN
+F 1 "KRL6432D-M-R006-G-T1" H 14450 5334 50  0000 C CNN
+F 2 "RESC3163X50N" H 14650 5250 50  0001 L CNN
+F 3 "http://www.mouser.com/datasheet/2/392/n_catalog_partition19_en-1114600.pdf" H 14650 5150 50  0001 L CNN
+F 4 "Current Sense Resistors - SMD 0.006 ohm 1% 3.0W" H 14650 5050 50  0001 L CNN "Description"
+F 5 "0.5" H 14650 4950 50  0001 L CNN "Height"
+F 6 "Susumu" H 14650 4850 50  0001 L CNN "Manufacturer_Name"
+F 7 "KRL6432E-C-R006-F-T1" H 14650 4750 50  0001 L CNN "Manufacturer_Part_Number"
+F 8 "" H 14650 4650 50  0001 L CNN "Arrow Part Number"
+F 9 "" H 14650 4550 50  0001 L CNN "Arrow Price/Stock"
+F 10 "754-KRL6432ECR006FT1" H 14650 4450 50  0001 L CNN "Mouser Part Number"
+F 11 "https://www.mouser.co.uk/ProductDetail/Susumu/KRL6432E-C-R006-F-T1/?qs=lc2O%252BfHJPVZeFQbLV4n%2Fcw%3D%3D" H 14650 4350 50  0001 L CNN "Mouser Price/Stock"
+	1    14100 5200
+	1    0    0    -1
+$EndComp
+$Comp
+L SamacSys_Parts:KRL6432E-C-R006-F-T1 R?
+U 1 1 5FFA1008
+P 14100 5450
+F 0 "R?" H 14450 5600 50  0000 C CNN
+F 1 "KRL6432D-M-R006-G-T1" H 14450 5550 50  0000 C CNN
+F 2 "RESC3163X50N" H 14650 5500 50  0001 L CNN
+F 3 "http://www.mouser.com/datasheet/2/392/n_catalog_partition19_en-1114600.pdf" H 14650 5400 50  0001 L CNN
+F 4 "Current Sense Resistors - SMD 0.006 ohm 1% 3.0W" H 14650 5300 50  0001 L CNN "Description"
+F 5 "0.5" H 14650 5200 50  0001 L CNN "Height"
+F 6 "Susumu" H 14650 5100 50  0001 L CNN "Manufacturer_Name"
+F 7 "KRL6432E-C-R006-F-T1" H 14650 5000 50  0001 L CNN "Manufacturer_Part_Number"
+F 8 "" H 14650 4900 50  0001 L CNN "Arrow Part Number"
+F 9 "" H 14650 4800 50  0001 L CNN "Arrow Price/Stock"
+F 10 "754-KRL6432ECR006FT1" H 14650 4700 50  0001 L CNN "Mouser Part Number"
+F 11 "https://www.mouser.co.uk/ProductDetail/Susumu/KRL6432E-C-R006-F-T1/?qs=lc2O%252BfHJPVZeFQbLV4n%2Fcw%3D%3D" H 14650 4600 50  0001 L CNN "Mouser Price/Stock"
+	1    14100 5450
+	1    0    0    -1
+$EndComp
+Wire Wire Line
+	14100 5200 14100 5450
+Wire Wire Line
+	14800 5200 14800 5450
+Wire Wire Line
+	14800 5450 14800 5800
+Connection ~ 14800 5450
+Connection ~ 14800 5800
+Wire Wire Line
+	14100 5450 14100 5800
+Connection ~ 14100 5450
+Connection ~ 14100 5800
 $EndSCHEMATC
