File: kicad/file5FD25DF8.sch (KiCad schematic (older format))
At the start: 18 parts, among them IC1 LD39100PU33R, J1 Screw_Terminal_01x02, U1 TPSM53604RDAR

Commit message: Power reg Section 1 initial entry; annotate
Parts:
- renumbered U1 to IC2
Changed lines of the file:
@@
 $EndComp
 $Comp
-L 2020-12-12_03-26-08:TPSM53604RDAR U1
+L 2020-12-12_03-26-08:TPSM53604RDAR IC2
 U 1 1 5FD45ECC
 P 5300 4450
-F 0 "U1" H 6100 4837 60  0000 C CNN
+F 0 "IC2" H 6100 4837 60  0000 C CNN
 F 1 "TPSM53604RDAR" H 6100 4731 60  0000 C CNN
 F 2 "B3QFN14_RDA_TEX" H 6100 4690 60  0001 C CNN

Commit message: Ethernet initial schematic; start ERC
Parts:
- renumbered IC2 to IC4, IC1 to IC5
Connections:
- net IC4FB: now reaches IC4.9 (FB), R2.2, R4.1
Other:
- moved on the sheet: C1, C2, C26, C27, C28, C3, C4, C5, D1, IC4, IC5, J1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

Commit message: Add datasheets
Parts:
- C26, C27, C28, C5: footprint (none) -> Capacitor_SMD:C_01005_0402Metric
- D1: footprint (none) -> LED_SMD:LED_0402_1005Metric
- L1: footprint IND_NLCV32T-R33M-PFR -> Inductor_SMD:L_0402_1005Metric
- R10, R3: footprint (none) -> Resistor_SMD:R_0402_1005Metric
Changed lines of the file:
@@
 $Descr USLedger 17000 11000
 encoding utf-8
-Sheet 2 6
+Sheet 2 5
 Title "KQ9P Power Controller 12VDC"
 Date "2020-12-08"
@@
 F 0 "L1" H 3350 4781 50  0000 C CNN
 F 1 "NLCV32T-R33M-EFR" H 3350 4690 50  0000 C CNN
-F 2 "IND_NLCV32T-R33M-PFR" H 3350 4600 50  0001 L BNN
+F 2 "Inductor_SMD:L_0402_1005Metric" H 3350 4600 50  0001 L BNN
 F 3 "" H 3350 4600 50  0001 L BNN
 F 4 "TDK" H 3350 4600 50  0001 L BNN "MANUFACTURER"
@@
 F 0 "R3" V 6595 3650 50  0000 C CNN
 F 1 "100k" V 6686 3650 50  0000 C CNN
-F 2 "" H 6800 3650 50  0001 C CNN
+F 2 "Resistor_SMD:R_0402_1005Metric" H 6800 3650 50  0001 C CNN
 F 3 "~" H 6800 3650 50  0001 C CNN
 	1    6800 3650
@@
 F 0 "C5" H 10915 5546 50  0000 L CNN
 F 1 "1uF_X5R" H 10915 5455 50  0000 L CNN
-F 2 "" H 10838 5350 50  0001 C CNN
+F 2 "Capacitor_SMD:C_01005_0402Metric" H 10838 5350 50  0001 C CNN
 F 3 "~" H 10800 5500 50  0001 C CNN
 	1    10800 5500
@@
 F 0 "C26" H 11365 5896 50  0000 L CNN
 F 1 "100nF" H 11365 5805 50  0000 L CNN
-F 2 "" H 11288 5700 50  0001 C CNN
+F 2 "Capacitor_SMD:C_01005_0402Metric" H 11288 5700 50  0001 C CNN
 F 3 "~" H 11250 5850 50  0001 C CNN
 	1    11250 5850
@@
 F 0 "C27" H 13165 6046 50  0000 L CNN
 F 1 "1uF_X5R" H 13165 5955 50  0000 L CNN
-F 2 "" H 13088 5850 50  0001 C CNN
+F 2 "Capacitor_SMD:C_01005_0402Metric" H 13088 5850 50  0001 C CNN
 F 3 "~" H 13050 6000 50  0001 C CNN
 	1    13050 6000
@@
 F 0 "C28" H 13765 5546 50  0000 L CNN
 F 1 "100nF" H 13765 5455 50  0000 L CNN
-F 2 "" H 13688 5350 50  0001 C CNN
+F 2 "Capacitor_SMD:C_01005_0402Metric" H 13688 5350 50  0001 C CNN
 F 3 "~" H 13650 5500 50  0001 C CNN
 	1    13650 5500
@@
 F 0 "D1" V 10439 5330 50  0000 L CNN
 F 1 "LED GREEN" V 10348 5330 50  0000 L CNN
-F 2 "" H 10400 5250 50  0001 C CNN
+F 2 "LED_SMD:LED_0402_1005Metric" H 10400 5250 50  0001 C CNN
 F 3 "~" H 10400 5250 50  0001 C CNN
 	1    10400 5250
@@
 F 0 "R10" H 10468 4896 50  0000 L CNN
 F 1 "1K" H 10468 4805 50  0000 L CNN
-F 2 "" H 10400 4850 50  0001 C CNN
+F 2 "Resistor_SMD:R_0402_1005Metric" H 10400 4850 50  0001 C CNN
 F 3 "~" H 10400 4850 50  0001 C CNN
 	1    10400 4850
