File: kicad/file5FD83A3A.sch (KiCad schematic (older format))
At the start: 30 parts, among them IC1 STM32F439VITx, J3 Conn_ARM_JTAG_SWD_10, SW1 RESET, Y1 NX3225GD-8.000M-EXS00A-CG04874

Commit message: Add datasheets
Parts:
- C10, C11, C12, C13, C14, C15, C17, C18, C19, C20, C21, C22, C23, C24, C25, C7: footprint (none) -> Capacitor_SMD:CP_Elec_4x5.4
- C16, C6, C8, C9: footprint (none) -> Capacitor_SMD:C_01005_0402Metric
- L2: footprint (none) -> Inductor_SMD:L_0402_1005Metric
- R5, R6, R7, R8, R9: footprint (none) -> Resistor_SMD:R_0402_1005Metric
- SW1: footprint (none) -> Button_Switch_SMD:SW_Push_1P1T_NO_6x6mm_H9.5mm
Changed lines of the file:
@@
 $Descr USLedger 17000 11000
 encoding utf-8
-Sheet 3 6
+Sheet 3 5
 Title "KQ9P Power Controller 12VDC"
 Date "2020-12-08"
@@
 F 0 "C19" H 9036 3454 50  0000 R CNN
 F 1 "10nF" H 9036 3545 50  0000 R CNN
-F 2 "" H 9150 3500 50  0001 C CNN
+F 2 "Capacitor_SMD:CP_Elec_4x5.4" H 9150 3500 50  0001 C CNN
 F 3 "~" H 9150 3500 50  0001 C CNN
 	1    9150 3500
@@
 F 0 "C22" H 9385 3454 50  0000 R CNN
 F 1 "1uF" H 9385 3545 50  0000 R CNN
-F 2 "" H 9500 3500 50  0001 C CNN
+F 2 "Capacitor_SMD:CP_Elec_4x5.4" H 9500 3500 50  0001 C CNN
 F 3 "~" H 9500 3500 50  0001 C CNN
 	1    9500 3500
@@
 F 0 "L2" H 9753 3546 50  0000 L CNN
 F 1 "22uH" H 9753 3455 50  0000 L CNN
-F 2 "" H 9700 3500 50  0001 C CNN
+F 2 "Inductor_SMD:L_0402_1005Metric" H 9700 3500 50  0001 C CNN
 F 3 "~" H 9700 3500 50  0001 C CNN
 	1    9700 3500
@@
 F 0 "C11" H 6785 2804 50  0000 R CNN
 F 1 "1uF" H 6785 2895 50  0000 R CNN
-F 2 "" H 6900 2850 50  0001 C CNN
+F 2 "Capacitor_SMD:CP_Elec_4x5.4" H 6900 2850 50  0001 C CNN
 F 3 "~" H 6900 2850 50  0001 C CNN
 	1    6900 2850
@@
 F 0 "C12" H 7136 2804 50  0000 R CNN
 F 1 "100nF" H 7136 2895 50  0000 R CNN
-F 2 "" H 7250 2850 50  0001 C CNN
+F 2 "Capacitor_SMD:CP_Elec_4x5.4" H 7250 2850 50  0001 C CNN
 F 3 "~" H 7250 2850 50  0001 C CNN
 	1    7250 2850
@@
 F 0 "C13" H 7385 2554 50  0000 R CNN
 F 1 "1uF" H 7385 2645 50  0000 R CNN
-F 2 "" H 7500 2600 50  0001 C CNN
+F 2 "Capacitor_SMD:CP_Elec_4x5.4" H 7500 2600 50  0001 C CNN
 F 3 "~" H 7500 2600 50  0001 C CNN
 	1    7500 2600
@@
 F 0 "C15" H 7736 2554 50  0000 R CNN
 F 1 "100nF" H 7736 2645 50  0000 R CNN
-F 2 "" H 7850 2600 50  0001 C CNN
+F 2 "Capacitor_SMD:CP_Elec_4x5.4" H 7850 2600 50  0001 C CNN
 F 3 "~" H 7850 2600 50  0001 C CNN
 	1    7850 2600
@@
 F 0 "C14" H 7485 1804 50  0000 R CNN
 F 1 "1uF" H 7485 1895 50  0000 R CNN
-F 2 "" H 7600 1850 50  0001 C CNN
+F 2 "Capacitor_SMD:CP_Elec_4x5.4" H 7600 1850 50  0001 C CNN
 F 3 "~" H 7600 1850 50  0001 C CNN
 	1    7600 1850
@@
 F 0 "C17" H 7836 1804 50  0000 R CNN
 F 1 "100nF" H 7836 1895 50  0000 R CNN
-F 2 "" H 7950 1850 50  0001 C CNN
+F 2 "Capacitor_SMD:CP_Elec_4x5.4" H 7950 1850 50  0001 C CNN
 F 3 "~" H 7950 1850 50  0001 C CNN
 	1    7950 1850
@@
 F 0 "C25" H 10085 2804 50  0000 R CNN
 F 1 "1uF" H 10085 2895 50  0000 R CNN
-F 2 "" H 10200 2850 50  0001 C CNN
+F 2 "Capacitor_SMD:CP_Elec_4x5.4" H 10200 2850 50  0001 C CNN
 F 3 "~" H 10200 2850 50  0001 C CNN
 	1    10200 2850
@@
 F 0 "C24" H 9736 2804 50  0000 R CNN
 F 1 "100nF" H 9736 2895 50  0000 R CNN
-F 2 "" H 9850 2850 50  0001 C CNN
+F 2 "Capacitor_SMD:CP_Elec_4x5.4" H 9850 2850 50  0001 C CNN
 F 3 "~" H 9850 2850 50  0001 C CNN
 	1    9850 2850
@@
 F 0 "C23" H 9485 2554 50  0000 R CNN
 F 1 "1uF" H 9485 2645 50  0000 R CNN
-F 2 "" H 9600 2600 50  0001 C CNN
+F 2 "Capacitor_SMD:CP_Elec_4x5.4" H 9600 2600 50  0001 C CNN
 F 3 "~" H 9600 2600 50  0001 C CNN
 	1    9600 2600
@@
 F 0 "C20" H 9136 2554 50  0000 R CNN
 F 1 "100nF" H 9136 2645 50  0000 R CNN
-F 2 "" H 9250 2600 50  0001 C CNN
+F 2 "Capacitor_SMD:CP_Elec_4x5.4" H 9250 2600 50  0001 C CNN
 F 3 "~" H 9250 2600 50  0001 C CNN
 	1    9250 2600
@@
 F 0 "C21" H 9385 1804 50  0000 R CNN
 F 1 "1uF" H 9385 1895 50  0000 R CNN
-F 2 "" H 9500 1850 50  0001 C CNN
+F 2 "Capacitor_SMD:CP_Elec_4x5.4" H 9500 1850 50  0001 C CNN
 F 3 "~" H 9500 1850 50  0001 C CNN
 	1    9500 1850
@@
 F 0 "C18" H 9036 1804 50  0000 R CNN
 F 1 "100nF" H 9036 1895 50  0000 R CNN
-F 2 "" H 9150 1850 50  0001 C CNN
+F 2 "Capacitor_SMD:CP_Elec_4x5.4" H 9150 1850 50  0001 C CNN
 F 3 "~" H 9150 1850 50  0001 C CNN
 	1    9150 1850
@@
 F 0 "SW1" H 5100 4485 50  0000 C CNN
 F 1 "RESET" H 5100 4394 50  0000 C CNN
-F 2 "" H 5100 4400 50  0001 C CNN
+F 2 "Button_Switch_SMD:SW_Push_1P1T_NO_6x6mm_H9.5mm" H 5100 4400 50  0001 C CNN
 F 3 "~" H 5100 4400 50  0001 C CNN
 	1    5100 4200
@@
 F 0 "C7" H 6265 6446 50  0000 L CNN
 F 1 "4.3pF" H 6265 6355 50  0000 L CNN
-F 2 "" H 6150 6400 50  0001 C CNN
+F 2 "Capacitor_SMD:CP_Elec_4x5.4" H 6150 6400 50  0001 C CNN
 F 3 "~" H 6150 6400 50  0001 C CNN
 	1    6150 6400
@@
 F 0 "C10" H 6765 6446 50  0000 L CNN
 F 1 "4.3pF" H 6765 6355 50  0000 L CNN
-F 2 "" H 6650 6400 50  0001 C CNN
+F 2 "Capacitor_SMD:CP_Elec_4x5.4" H 6650 6400 50  0001 C CNN
 F 3 "~" H 6650 6400 50  0001 C CNN
 	1    6650 6400
@@
 F 0 "R8" V 6100 4250 50  0000 C CNN
 F 1 "100K" V 6200 4250 50  0000 C CNN
-F 2 "" H 6000 4250 50  0001 C CNN
+F 2 "Resistor_SMD:R_0402_1005Metric" H 6000 4250 50  0001 C CNN
 F 3 "~" H 6000 4250 50  0001 C CNN
 	1    6000 4250
@@
 F 0 "C8" V 6371 4600 50  0000 C CNN
 F 1 "2.2uF" V 6462 4600 50  0000 C CNN
-F 2 "" H 6600 4600 50  0001 C CNN
+F 2 "Capacitor_SMD:C_01005_0402Metric" H 6600 4600 50  0001 C CNN
 F 3 "~" H 6600 4600 50  0001 C CNN
 	1    6600 4600
@@
 F 0 "C9" V 6371 5000 50  0000 C CNN
 F 1 "2.2uF" V 6462 5000 50  0000 C CNN
-F 2 "" H 6600 5000 50  0001 C CNN
+F 2 "Capacitor_SMD:C_01005_0402Metric" H 6600 5000 50  0001 C CNN
 F 3 "~" H 6600 5000 50  0001 C CNN
 	1    6600 5000
@@
 F 0 "C6" V 4848 4700 50  0000 C CNN
 F 1 "100nF" V 4939 4700 50  0000 C CNN
-F 2 "" H 5138 4550 50  0001 C CNN
+F 2 "Capacitor_SMD:C_01005_0402Metric" H 5138 4550 50  0001 C CNN
 F 3 "~" H 5100 4700 50  0001 C CNN
 	1    5100 4700
@@
 F 0 "C16" V 7648 3750 50  0000 C CNN
 F 1 "C" V 7739 3750 50  0000 C CNN
-F 2 "" H 7938 3600 50  0001 C CNN
+F 2 "Capacitor_SMD:C_01005_0402Metric" H 7938 3600 50  0001 C CNN
 F 3 "~" H 7900 3750 50  0001 C CNN
 	1    7900 3750
@@
 F 0 "R9" H 11618 6546 50  0000 L CNN
 F 1 "10k" H 11618 6455 50  0000 L CNN
-F 2 "" H 11550 6500 50  0001 C CNN
+F 2 "Resistor_SMD:R_0402_1005Metric" H 11550 6500 50  0001 C CNN
 F 3 "~" H 11550 6500 50  0001 C CNN
 	1    11550 6500
@@
 F 0 "R7" H 11368 6546 50  0000 L CNN
 F 1 "10k" H 11368 6455 50  0000 L CNN
-F 2 "" H 11300 6500 50  0001 C CNN
+F 2 "Resistor_SMD:R_0402_1005Metric" H 11300 6500 50  0001 C CNN
 F 3 "~" H 11300 6500 50  0001 C CNN
 	1    11300 6500
@@
 F 0 "R6" H 11118 6546 50  0000 L CNN
 F 1 "10k" H 11118 6455 50  0000 L CNN
-F 2 "" H 11050 6500 50  0001 C CNN
+F 2 "Resistor_SMD:R_0402_1005Metric" H 11050 6500 50  0001 C CNN
 F 3 "~" H 11050 6500 50  0001 C CNN
 	1    11050 6500
@@
 F 0 "R5" H 10868 6546 50  0000 L CNN
 F 1 "10k" H 10868 6455 50  0000 L CNN
-F 2 "" H 10800 6500 50  0001 C CNN
+F 2 "Resistor_SMD:R_0402_1005Metric" H 10800 6500 50  0001 C CNN
 F 3 "~" H 10800 6500 50  0001 C CNN
 	1    10800 6500
