File: kicad/file5FD26A29.sch (KiCad schematic (older format))
At the start: 37 parts, among them IC3 USBLC6-4SC6, J2 6339191-4, T1 H1102NLT, U3 LAN8742A-CZ-TR, Y2 SXT3249AA17-25.000M

Commit message: Add datasheets
Parts:
- C29, C30, C31, C83, C84, C85, C86, C87, C88: footprint (none) -> Capacitor_SMD:C_01005_0402Metric
- FB1: footprint (none) -> Ferrite_THT:LairdTech_28C0236-0JW-10
- R41, R42, R43, R44, R45, R46, R47, R48, R49, R50, R51, R52, R53, R54, R55, R56, R57, R58, R59, R60, R61: footprint (none) -> Resistor_SMD:R_0402_1005Metric

Commit message: Finalize parts change, separate regulator to separate project
Connections:
- net +3V3: now also C29.1, C30.1, C31.1, C86.1, C88.1, T1.2, T1.7, U3.1 (VDD2A), U3.19 (VDD1A)
Changed lines of the file:
@@
 	8250 5650 9200 5650
 Wire Wire Line
-	9200 5650 9200 6350
+	9200 5650 9200 5900
 Wire Wire Line
 	9200 7350 8100 7350
@@
 Wire Wire Line
 	3150 5550 3650 5550
+$Comp
+L power:+3V3 #PWR?
+U 1 1 5FEAC77A
+P 9300 5900
+F 0 "#PWR?" H 9300 5750 50  0001 C CNN
+F 1 "+3V3" V 9315 6028 50  0000 L CNN
+F 2 "" H 9300 5900 50  0001 C CNN
+F 3 "" H 9300 5900 50  0001 C CNN
+	1    9300 5900
+	0    1    1    0
+$EndComp
+Wire Wire Line
+	9300 5900 9200 5900
+Connection ~ 9200 5900
+Wire Wire Line
+	9200 5900 9200 6350
 $EndSCHEMATC
